File: entangler/hardware/entangler.kicad_pcb (KiCad board)
At the start: 2 copper layers, 39 x 28 mm, 7 parts, among them J1 Conn_01x03_Pin, J2 USB_C_Receptacle, J3 Conn_01x02_Pin, U1 RP2040, U2 MCP73831-2-MC, U3 AP2112K-3.3

Commit message: Progress towards v0.2
Parts:
- removed U1: RP2040, Package_DFN_QFN:QFN-56-1EP_7x7mm_P0.4mm_EP3.2x3.2mm
- removed the U3 at (132.4, 114.5)
- added C1: 100nf, Capacitor_SMD:C_0402_1005Metric, F.Cu at (222.1, 103.3)
- added C10: 2.2uf, Capacitor_SMD:C_0402_1005Metric, F.Cu at (214.1, 128.0)
- added C10: 2.2uf, Capacitor_SMD:C_0402_1005Metric, F.Cu at (225.0, 109.2)
- added C11: 100nf, Capacitor_SMD:C_0402_1005Metric, F.Cu at (225.0, 111.2)
- added C11: 100nf, Capacitor_SMD:C_0402_1005Metric, F.Cu at (214.1, 130.0)
- added C12: 100nf, Capacitor_SMD:C_0402_1005Metric, F.Cu at (225.0, 113.2)
- added C12: 100nf, Capacitor_SMD:C_0402_1005Metric, F.Cu at (214.1, 132.0)
- added C13: 10uf, Capacitor_SMD:C_0402_1005Metric, F.Cu at (227.9, 103.3)
- added C14: 100nf, Capacitor_SMD:C_0402_1005Metric, F.Cu at (227.9, 105.3)
- added C15: 10uf, Capacitor_SMD:C_0402_1005Metric, F.Cu at (227.9, 107.3)
- added C2: 22uf, Capacitor_SMD:C_0402_1005Metric, F.Cu at (222.1, 105.3)
- added C3: 22uf, Capacitor_SMD:C_0402_1005Metric, F.Cu at (222.1, 107.3)
- added C4: 10uf, Capacitor_SMD:C_0402_1005Metric, F.Cu at (222.1, 109.2)
- added C5: 15pf, Capacitor_SMD:C_0402_1005Metric, F.Cu at (214.1, 118.2)
- added C5: 15pf, Capacitor_SMD:C_0402_1005Metric, F.Cu at (222.1, 111.2)
- added C6: 15pf, Capacitor_SMD:C_0402_1005Metric, F.Cu at (222.1, 113.2)
- added C6: 15pf, Capacitor_SMD:C_0402_1005Metric, F.Cu at (214.1, 120.1)
- added C7: 2.2uf, Capacitor_SMD:C_0402_1005Metric, F.Cu at (225.0, 103.3)
- added C7: 2.2uf, Capacitor_SMD:C_0402_1005Metric, F.Cu at (214.1, 122.1)
- added C8: 100nf, Capacitor_SMD:C_0402_1005Metric, F.Cu at (225.0, 105.3)
- added C8: 100nf, Capacitor_SMD:C_0402_1005Metric, F.Cu at (214.1, 124.1)
- added C9: 100nf, Capacitor_SMD:C_0402_1005Metric, F.Cu at (225.0, 107.3)
- added C9: 100nf, Capacitor_SMD:C_0402_1005Metric, F.Cu at (214.1, 126.0)
- added D1: LED, LED_SMD:LED_0603_1608Metric, F.Cu at (225.9, 95.4)
- added D3: LED, LED_SMD:LED_0603_1608Metric, F.Cu at (225.9, 100.6)
- added L1: 10uh, Inductor_SMD:L_TDK_NLV32_3.2x2.5mm, F.Cu at (232.3, 113.8)
- added P1: S2B-PH-SM4-TB, S2B-PH-SM4-TB:JST_S2B-PH-SM4-TB, F.Cu at (112.5, 107.9)
- added R1: 5.1kr, Resistor_SMD:R_0402_1005Metric, F.Cu at (202.9, 128.8)
- added R10: 1kr, Resistor_SMD:R_0402_1005Metric, F.Cu at (222.4, 99.7)
- added R10: 1kr, Resistor_SMD:R_0402_1005Metric, F.Cu at (217.0, 132.2)
- added R2: 5.1kr, Resistor_SMD:R_0402_1005Metric, F.Cu at (202.9, 130.8)
- added R3: 27r, Resistor_SMD:R_0402_1005Metric, F.Cu at (217.0, 126.2)
- added R3: 27r, Resistor_SMD:R_0402_1005Metric, F.Cu at (222.4, 85.8)
- added R4: 27r, Resistor_SMD:R_0402_1005Metric, F.Cu at (217.0, 128.2)
- added R4: 27r, Resistor_SMD:R_0402_1005Metric, F.Cu at (222.4, 87.8)
- added R5: 66.5r, Resistor_SMD:R_0402_1005Metric, F.Cu at (222.4, 89.8)
- added R6: 66.5r, Resistor_SMD:R_0402_1005Metric, F.Cu at (222.4, 91.8)
- added R7: 10kr, Resistor_SMD:R_0402_1005Metric, F.Cu at (222.4, 93.7)
- added R8: 66.5r, Resistor_SMD:R_0402_1005Metric, F.Cu at (222.4, 95.7)
- added R9: 1kr, Resistor_SMD:R_0402_1005Metric, F.Cu at (217.0, 130.2)
- added R9: 1kr, Resistor_SMD:R_0402_1005Metric, F.Cu at (222.4, 97.7)
- added SW1: Push_Button, Button_Switch_SMD:SW_SPST_PTS810, F.Cu at (111.5, 121.5)
- added SW1: Push_Button, Button_Switch_SMD:SW_SPST_PTS810, F.Cu at (117.5, 121.5)
- added U3: RP2040, Package_DFN_QFN:QFN-56-1EP_7x7mm_P0.4mm_EP3.2x3.2mm, F.Cu at (228.5, 89.4)
- added U3: LC86G, LC86G:XCVR_LC86G, F.Cu at (150.0, 112.5)
- added U4: AP63203WU, Package_TO_SOT_SMD:TSOT-23-6, F.Cu at (231.9, 109.5)
- added U5: W25Q32JVZP, Package_SON:WSON-8-1EP_6x5mm_P1.27mm_EP3.4x4.3mm, F.Cu at (223.8, 120.5)
- added U5: W25Q32JVZP, Package_SON:WSON-8-1EP_6x5mm_P1.27mm_EP3.4x4.3mm, F.Cu at (232.2, 97.4)
- D2: value MBR1020VL -> LED; footprint Diode_SMD:D_SOD-123F -> LED_SMD:LED_0603_1608Metric
- J1: value Conn_01x03_Pin -> Conn_Coaxial_Small; footprint Connector_PinSocket_2.00mm:PinSocket_1x03_P2.00mm_Vertical -> Connector_Coaxial:SMA_Amphenol_132289_EdgeMount
- J2: value USB_C_Receptacle -> Conn_01x03; footprint Connector_USB:USB_C_Receptacle_GCT_USB4105-xx-A_16P_TopMnt_Horizontal -> Connector_PinHeader_2.00mm:PinHeader_1x03_P2.00mm_Vertical
- J3: value Conn_01x02_Pin -> USB-7010ASV; footprint Connector_JST:JST_PH_B2B-PH-SM4-TB_1x02-1MP_P2.00mm_Vertical -> Connector_USB:USB_C_Receptacle_G-Switch_GT-USB-7010ASV
- U2: value MCP73831-2-MC -> RFM95W-868S2; footprint Package_DFN_QFN:DFN-8-1EP_3x2mm_P0.5mm_EP1.7x1.4mm -> RF_Module:HOPERF_RFM9XW_SMD; moved to B.Cu
- moved D2 99.6 mm to (225.9, 98.0)
- moved J2 84.5 mm to (217.5, 119.2)
- moved J1 49.0 mm to (168.6, 112.5)
- moved U2 25.9 mm to (153.0, 112.5), turned to -90 degrees
- moved J3 11.3 mm to (103.0, 112.5), turned to -90 degrees
Connections:
- D2 pad 1: /Power/VBUS -> GND
- D2 pad 2: /Power/VBAT -> Net-(D2-A)
- J1 pad 1: GND -> Net-(J1-In)
- J1 pad 2: Net-(J1-Pin_2) -> GND
- U2 pad 1: /Power/VBUS -> GND
- U2 pad 2: /Power/VBUS -> MISO
- U2 pad 3: /Power/VBAT -> MOSI
- U2 pad 4: /Power/VBAT -> SCK
- U2 pad 5: Net-(U2-STAT) -> CSN
- U2 pad 6: GND -> RF_RST
- U2 pad 8: Net-(U2-PROG) -> GND
- U2 pad 9: (no net) -> Net-(J1-In)
Routing:
- net GND: track 0.00 -> 5.37 mm
Other:
- board size 39 x 28 mm -> 71.5 x 25 mm
- copper layers 2 -> 4
- board text added: "By Tim Gibson"
- board text added: "Entangler v1"
