File: entangler/hardware/entangler.kicad_sch (KiCad schematic)
At the start: 5 parts, among them J1 Conn_01x03_Pin, J3 Conn_01x02_Pin, U1 RP2040

Commit message: Progress towards v0.2
Parts:
- removed J1: Conn_01x03_Pin, Connector_PinSocket_2.00mm:PinSocket_1x03_P2.00mm_Vertical, symbol Connector:Conn_01x03_Pin
- removed J3: Conn_01x02_Pin, Connector_JST:JST_PH_B2B-PH-SM4-TB_1x02-1MP_P2.00mm_Vertical, symbol Connector:Conn_01x02_Pin
- removed U1: RP2040, Package_DFN_QFN:QFN-56-1EP_7x7mm_P0.4mm_EP3.2x3.2mm, symbol MCU_RaspberryPi:RP2040
- added C1, C14: 100nf, Capacitor_SMD:C_0402_1005Metric, symbol Device:C
- added C13, C15, C4: 10uf, Capacitor_SMD:C_0402_1005Metric, symbol Device:C
- added C2, C3: 22uf, Capacitor_SMD:C_0402_1005Metric, symbol Device:C
- added D1, D2, D3: LED, LED_SMD:LED_0603_1608Metric, symbol Device:LED
- added J1: Conn_Coaxial_Small, Connector_Coaxial:SMA_Amphenol_132289_EdgeMount, symbol Connector:Conn_Coaxial_Small
- added L1: 10uh, Inductor_SMD:L_TDK_NLV32_3.2x2.5mm, symbol Device:L
- added P1: S2B-PH-SM4-TB, S2B-PH-SM4-TB:JST_S2B-PH-SM4-TB, symbol JST-PH-2:S2B-PH-SM4-TB
- added R5, R8: 66.5r, Resistor_SMD:R_0402_1005Metric, symbol Device:R
- added U2: RFM95W-868S2, RF_Module:HOPERF_RFM9XW_SMD, symbol RF_Module:RFM95W-868S2
- added U3: LC86G, LC86G:XCVR_LC86G, symbol LC86G:LC86G
- added U4: AP63203WU, Package_TO_SOT_SMD:TSOT-23-6, symbol Regulator_Switching:AP63203WU
- R6: value 27 -> 66.5r; footprint (none) -> Resistor_SMD:R_0402_1005Metric; DESCRIPTION (none) -> ERJ-3EKF66R5V
- R7: value 27 -> 10kr; footprint (none) -> Resistor_SMD:R_0402_1005Metric; DESCRIPTION (none) -> ERJ-3EKF1002V
Connections:
- net USB_DM is gone; now on net +3V3: R7.1
- net +3V3: now also C13.1, C14.1, C15.1, C2.2, C3.2, L1.2, R5.1, U2.13 (3.3V), U3.4 (VCC), U3.5 (V_BCKP), U4.1 (FB)
- net GND: now also C13.2, C14.2, C15.2, C2.1, C3.1, C4.2, D1.1 (K), D2.1 (K), D3.1 (K), J1.2 (Ext), P1.2, U2.1 (GND), U2.10 (GND), U2.8 (GND), U3.12 (GND), U3.13 (GND), U3.14 (GND), U3.15 (GND), U3.16 (GND), U3.17 (GND), U3.18 (GND), U3.19 (GND), U3.20 (GND), U3.21 (GND), U3.22 (GND), U3.23 (GND), U3.24 (GND), U3.25 (GND), U3.26 (GND), U3.27 (GND), U3.28 (GND), U3.29 (GND), U3.3 (GND), U3.30 (GND), U3.31 (GND), U3.32 (GND), U3.33 (GND), U3.34 (GND), U3.35 (GND), U3.36 (GND), U4.4 (GND)
- net GPS_RST: now reaches R7.2
- net GPS_RST: now also U3.10 (~{RESET})
- net at R6.2: now also D2.2 (A)
- net USB_DP renamed LED_1
- new net: C1.2, L1.1, U4.6 (BST)
- new net: U3.7 (RESERVED), U3.9 (RESERVED)
- new net: D3.2 (A), R8.2
- new net: J1.1 (In), U2.9 (ANT)
- new net: D1.2 (A), R5.2
- new net: C1.1, U4.5 (SW)
- new net CSN: U2.5 (NSS)
- new net GPS_1PPS: R8.1, U3.6 (1PPS)
- new net MCU_RX: U3.2 (TXD)
- new net MCU_TX: U3.1 (RXD)
- new net MISO: U2.2 (MISO)
- new net MOSI: U2.3 (MOSI)
- new net RF_DIO: U2.14 (DIO0)
- new net RF_RST: U2.6 (RESET)
- new net SCK: U2.4 (SCK)
- new net VBAT: C4.1, P1.1, U4.2 (EN), U4.3 (IN)
- no-connect marks 0 -> 8
Other:
- removed sheet Power
- added sheet MCU (mcu.kicad_sch)

Commit message: Update libs + adding more pins
Parts:
- removed C1: 100nf, Capacitor_SMD:C_0402_1005Metric, symbol Device:C
- removed C2, C3: 22uf, Capacitor_SMD:C_0402_1005Metric, symbol Device:C
- removed C4: 10uf, Capacitor_SMD:C_0402_1005Metric, symbol Device:C
- removed L1: 10uh, Inductor_SMD:L_TDK_NLV32_3.2x2.5mm, symbol Device:L
- removed P1: S2B-PH-SM4-TB, S2B-PH-SM4-TB:JST_S2B-PH-SM4-TB, symbol JST-PH-2:S2B-PH-SM4-TB
- removed U4: AP63203WU, Package_TO_SOT_SMD:TSOT-23-6, symbol Regulator_Switching:AP63203WU
- added D4: PMEG2020EH, Diode_SMD:D_SOD-123F, symbol Diode:PMEG2020EH
- added P1: S2B-PH-SM4-TB, S2B-PH-SM4-TB:JST_S2B-PH-SM4-TB, symbol S2B-PH-SM4-TB:S2B-PH-SM4-TB
- added R9: 1kr, Resistor_SMD:R_0402_1005Metric, symbol Device:R
- added SW1: Push_Button, Button_Switch_SMD:SW_SPST_PTS810, symbol PCM_SL_Devices:Push_Button
- added U5: W25Q32JVZP, Package_SON:WSON-8-1EP_6x5mm_P1.27mm_EP3.4x4.3mm, symbol Memory_Flash:W25Q32JVZP
- D1, D2, D3: footprint LED_SMD:LED_0603_1608Metric -> LED_SMD:LED_0201_0603Metric; DESCRIPTION 150060RS75000 -> (none)
Connections:
- net +3V3: now also U5.8 (VCC)
- net GND: now also P1.2, SW1.1, U5.4 (GND)
- net CSN renamed RF_CSN
- net MCU_RX renamed GPS_TX
- net MCU_TX renamed GPS_RX
- net MISO renamed RF_MISO
- net MOSI renamed RF_MOSI
- net RF_DIO renamed RF_DIO_0
- net SCK renamed RF_SCK
- new net: R9.2, SW1.2
- new net BCC/VBAT: P1.1
- new net BCC/VBUS: D4.1 (K)
- new net QSPI_SCLK: U5.6 (CLK)
- new net QSPI_SD0: U5.5 (DI/IO_{0})
- new net QSPI_SD1: U5.2 (DO/IO_{1})
- new net QSPI_SD2: U5.3 (~{WP}/IO_{2})
- new net QSPI_SD3: U5.7 (~{HOLD}/~{RESET}/IO_{3})
- new net QSPI_SS: R9.1, U5.1 (~{CS})
- new net USB C/VBUS: D4.2 (A)
Other:
- added sheet BCC (BCS.kicad_sch)
- sheet MCU ports: added GPIO_2_GPS_RST, LED_1, QPSI_SS, QSPI_SCLK, QSPI_SD0, QSPI_SD1, QSPI_SD2, QSPI_SD3, RF_DIO, RF_RST, SPI_PRI_CS, SPI_PRI_MISO, SPI_PRI_MOSI, SPI_PRI_SCK, USART_PRI_RX, USART_PRI_TX, USB_DM, USB_DP; removed none
- moved on the sheet: C13, C14, C15, J1, R7, U2, U3
