File: entangler/hardware/mcu.kicad_sch (KiCad schematic)
At the start: 18 parts, among them J2 Conn_01x03, SW1 Push_Button, U5 W25Q32JVZP, U6 RP2350B-QFN80, Y1 ECS-120-20-33-AEL-TR

Commit message: Update libs + adding more pins
Parts:
- removed R9: 1kr, Resistor_SMD:R_0402_1005Metric, symbol Device:R
- removed SW1: Push_Button, Button_Switch_SMD:SW_SPST_PTS810, symbol PCM_SL_Devices:Push_Button
- removed U5: W25Q32JVZP, Package_SON:WSON-8-1EP_6x5mm_P1.27mm_EP3.4x4.3mm, symbol Memory_Flash:W25Q32JVZP
- removed U6: RP2350B-QFN80, symbol RP2350B:RP2350B-QFN80
- added R11: 10kr, symbol Device:R
- added U4: RP2350B-QFN80, symbol RP2350:RP2350B-QFN80
Connections:
- net +1V1: now also U4.10 (DVDD), U4.32 (DVDD), U4.51 (DVDD)
- net +3V3: now also R11.1
- net GND: now also U4.81 (GND)
- net GPIO_2_GPS_RST: now also U4.79 (GPIO2)
- net LED_1: now also U4.26 (GPIO25)
- net QSPI_SCLK: now also U4.71 (QSPI_SCLK)
- net QSPI_SD0: now also U4.72 (QSPI_SD0)
- net QSPI_SD1: now also U4.74 (QSPI_SD1)
- net QSPI_SD2: now also U4.73 (QSPI_SD2)
- net QSPI_SD3: now also U4.70 (QSPI_SD3)
- net RF_DIO: now also U4.2 (GPIO5)
- net RF_RST: now also U4.4 (GPIO7)
- net SPI_PRI_CS: now also U4.17 (GPIO17)
- net SPI_PRI_MISO: now also U4.16 (GPIO16)
- net SPI_PRI_MOSI: now also U4.19 (GPIO19)
- net SPI_PRI_SCK: now also U4.18 (GPIO18)
- net USART_PRI_RX: now also U4.78 (GPIO1)
- net USART_PRI_TX: now also U4.77 (GPIO0)
- net XIN: now also U4.30 (XIN)
- net XOUT: now also U4.31 (XOUT)
- net at J2.1 (Pin_1): now also U4.33 (SWCLK)
- net at J2.3 (Pin_3): now also U4.34 (SWDIO)
- net at L2.2: now also U4.63 (VREG_LX)
- net at R4.2: now also U4.66 (USB_DM)
- net at R3.2: now also U4.67 (USB_DP)
- new net: R11.2, U4.35 (RUN)
- new net QPSI_SS: U4.75 (QSPI_SS)
- no-connect marks 2 -> 48
Other:
- moved on the sheet: C5, C6, R10, Y1
