File: entangler/hardware/usb-c.kicad_sch (KiCad schematic)
At the start: 3 parts, among them J2 USB_C_Receptacle

Commit message: Progress towards v0.2
Parts:
- removed J2: USB_C_Receptacle, Connector_USB:USB_C_Receptacle_GCT_USB4105-xx-A_16P_TopMnt_Horizontal, symbol Connector:USB_C_Receptacle
- removed R4, R5: 5.1k, symbol Device:R
- added J3: USB-7010ASV, Connector_USB:USB_C_Receptacle_G-Switch_GT-USB-7010ASV, symbol Connector:USB_C_Receptacle_USB2.0_14P
- added R1, R2: 5.1kr, Resistor_SMD:R_0402_1005Metric, symbol Device:R
Connections:
- net GND: now also J3.A1 (GND), J3.A12 (GND), J3.B1 (GND), J3.B12 (GND), R1.2, R2.2
- net USB_DM: now also J3.A7 (D-), J3.B7 (D-)
- net USB_DP: now also J3.A6 (D+), J3.B6 (D+)
- net VBUS: now also J3.A4 (VBUS), J3.A9 (VBUS), J3.B4 (VBUS), J3.B9 (VBUS)
- new net: J3.A5 (CC1), R1.1
- new net: J3.B5 (CC2), R2.1
- no-connect marks 10 -> 1

Commit message: Update libs + adding more pins
Changed lines of the file:
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@@
 	)
 	(hierarchical_label "USB_DP"
-		(shape input)
+		(shape passive)
 		(at 149.86 95.25 0)
 		(effects
@@
 	)
 	(hierarchical_label "VBUS"
-		(shape input)
+		(shape output)
 		(at 146.05 74.93 0)
 		(effects
@@
 	)
 	(hierarchical_label "USB_DM"
-		(shape input)
+		(shape passive)
 		(at 149.86 90.17 0)
 		(effects
@@
 		(instances
 			(project "entangler"
-				(path "/4b7f53f4-57b9-4873-88d3-e26b51eb832b/784eece9-66d1-4adf-8604-61719dcabce2"
+				(path "/4b7f53f4-57b9-4873-88d3-e26b51eb832b/fd15bdc7-b0bd-4057-872a-7c903c2848ee"
 					(reference "#PWR05")
 					(unit 1)
@@
 		(instances
 			(project "entangler"
-				(path "/4b7f53f4-57b9-4873-88d3-e26b51eb832b/784eece9-66d1-4adf-8604-61719dcabce2"
+				(path "/4b7f53f4-57b9-4873-88d3-e26b51eb832b/fd15bdc7-b0bd-4057-872a-7c903c2848ee"
 					(reference "#PWR06")
 					(unit 1)
@@
 		(instances
 			(project "entangler"
-				(path "/4b7f53f4-57b9-4873-88d3-e26b51eb832b/784eece9-66d1-4adf-8604-61719dcabce2"
+				(path "/4b7f53f4-57b9-4873-88d3-e26b51eb832b/fd15bdc7-b0bd-4057-872a-7c903c2848ee"
 					(reference "J3")
 					(unit 1)
@@
 		(instances
 			(project "entangler"
-				(path "/4b7f53f4-57b9-4873-88d3-e26b51eb832b/784eece9-66d1-4adf-8604-61719dcabce2"
+				(path "/4b7f53f4-57b9-4873-88d3-e26b51eb832b/fd15bdc7-b0bd-4057-872a-7c903c2848ee"
 					(reference "R2")
 					(unit 1)
@@
 		(instances
 			(project "entangler"
-				(path "/4b7f53f4-57b9-4873-88d3-e26b51eb832b/784eece9-66d1-4adf-8604-61719dcabce2"
+				(path "/4b7f53f4-57b9-4873-88d3-e26b51eb832b/fd15bdc7-b0bd-4057-872a-7c903c2848ee"
 					(reference "R1")
 					(unit 1)
